File: hardware/kicad/matrix-dev/matrix-dev-board.sch (KiCad schematic (older format))
At the start: 0 parts

Commit message: [ci skip] Schematic capture for a basic dev board based on the app circuit in the datasheet
Parts:
- added C? (x7): C, symbol C
- added J?: CONN_01X12, symbol CONN_01X12
- added J?: CONN_01X16, symbol CONN_01X16
- added J?: CONN_01X04, symbol CONN_01X04
- added J?: CONN_01X01, symbol CONN_01X01
- added J?: Screw_Terminal_1x02, symbol Screw_Terminal_1x02
- added R? (x10): R, symbol R
- added U?: IS31FL3733, symbol IS31FL3733
Connections:
- new net: J?.8 (P8), U?.10 (SW8)
- new net: J?.9 (P9), U?.11 (SW9)
- new net: J?.10 (P10), U?.13 (SW10)
- new net: J?.11 (P11), U?.14 (SW11)
- new net: J?.12 (P12), U?.15 (SW12)
- new net: J?.1 (P1), U?.16 (CS1)
- new net: J?.2 (P2), U?.17 (CS2)
- new net: J?.3 (P3), U?.18 (CS3)
- new net: J?.4 (P4), U?.19 (CS4)
- new net: J?.1 (P1), U?.2 (SW1)
- new net: J?.5 (P5), U?.21 (CS5)
- new net: J?.6 (P6), U?.22 (CS6)
- new net: J?.7 (P7), U?.23 (CS7)
- new net: J?.8 (P8), U?.24 (CS8)
- new net: J?.9 (P9), U?.25 (CS9)
- new net: J?.10 (P10), U?.26 (CS10)
- new net: J?.11 (P11), U?.27 (CS11)
- new net: J?.12 (P12), U?.28 (CS12)
- new net: J?.2 (P2), U?.3 (SW2)
- new net: J?.13 (P13), U?.30 (CS13)
- new net: J?.14 (P14), U?.31 (CS14)
- new net: J?.15 (P15), U?.32 (CS15)
- new net: J?.16 (P16), U?.33 (CS16)
- new net: R?.1, U?.35 (RSET)
- new net: J?.3 (P3), U?.4 (SW3)
- new net: J?.1 (P1), U?.40 (SYNC)
- new net: R?.1, U?.42 (SCL)
- new net: R?.1, U?.43 (ADDR1)
- new net: R?.1, U?.44 (ADDR2)
- new net: R?.1, U?.47 (IICRST)
- new net: J?.4 (P4), U?.6 (SW4)
- new net: J?.5 (P5), U?.7 (SW5)
- new net: J?.6 (P6), U?.8 (SW6)
- new net: J?.7 (P7), U?.9 (SW7)
- new net +3V3: C?.1, C?.2, C?.2, C?.2, C?.2, C?.2, C?.2, J?.1, J?.1 (P1), J?.2 (P2), J?.3 (P3), J?.4 (P4), R?.2, R?.2, R?.2, R?.2, R?.2, R?.2, U?.20 (PVCC), U?.29 (PVCC), U?.37 (AVCC), U?.38 (DVCC), U?.39 (VIO)
- new net GND: C?.1, C?.1, C?.1, C?.1, C?.1, C?.1, C?.2, J?.2, R?.1, R?.1, R?.2, R?.2, R?.2, R?.2, U?.12 (PGND), U?.34 (AGND), U?.48 (GND), U?.49 (PAD), U?.5 (PGND)

Commit message: [ci skip] Fix pull-up and pull-down resistors and add values
Parts:
- C? (x4): value C -> 0.47u
- C? (x3): value C -> 0.1u
- R? (x4): value R -> 0
- R? (x2): value R -> 1K
- R? (x3): value R -> 100K
- R?: value R -> 20K
Connections:
- net +3V3: no longer J?.1 (P1), J?.2 (P2), J?.3 (P3), J?.4 (P4), R?.2
- net GND: now also R?.1
- net at U?.41 (SDA): now also J?.1 (P1), R?.1
- net at U?.42 (SCL): now also J?.2 (P2), R?.1; no longer R?.1
- net at U?.45 (INTB): now also J?.3 (P3), R?.1
- net at U?.46 (SDB): now also J?.4 (P4), R?.2
Other:
- moved on the sheet: J?, R?
Changed lines of the file:
@@
 P 4700 5150
 F 0 "R?" V 4780 5150 50  0000 C CNN
-F 1 "R" V 4700 5150 50  0000 C CNN
+F 1 "0" V 4700 5150 50  0000 C CNN
 F 2 "" V 4630 5150 50  0001 C CNN
 F 3 "" H 4700 5150 50  0001 C CNN
@@
 P 4700 5500
 F 0 "R?" V 4780 5500 50  0000 C CNN
-F 1 "R" V 4700 5500 50  0000 C CNN
+F 1 "0" V 4700 5500 50  0000 C CNN
 F 2 "" V 4630 5500 50  0001 C CNN
 F 3 "" H 4700 5500 50  0001 C CNN
@@
 P 4300 5150
 F 0 "R?" V 4380 5150 50  0000 C CNN
-F 1 "R" V 4300 5150 50  0000 C CNN
+F 1 "0" V 4300 5150 50  0000 C CNN
 F 2 "" V 4230 5150 50  0001 C CNN
 F 3 "" H 4300 5150 50  0001 C CNN
@@
 P 4300 5500
 F 0 "R?" V 4380 5500 50  0000 C CNN
-F 1 "R" V 4300 5500 50  0000 C CNN
+F 1 "0" V 4300 5500 50  0000 C CNN
 F 2 "" V 4230 5500 50  0001 C CNN
 F 3 "" H 4300 5500 50  0001 C CNN
@@
 L R R?
 U 1 1 5AA9DEC1
-P 4600 3750
-F 0 "R?" V 4680 3750 50  0000 C CNN
-F 1 "R" V 4600 3750 50  0000 C CNN
-F 2 "" V 4530 3750 50  0001 C CNN
-F 3 "" H 4600 3750 50  0001 C CNN
-	1    4600 3750
-	0    1    1    0
+P 4150 3100
+F 0 "R?" V 4230 3100 50  0000 C CNN
+F 1 "1K" V 4150 3100 50  0000 C CNN
+F 2 "" V 4080 3100 50  0001 C CNN
+F 3 "" H 4150 3100 50  0001 C CNN
+	1    4150 3100
+	-1   0    0    1
 $EndComp
 $Comp
 L R R?
 U 1 1 5AA9E017
-P 4600 3450
-F 0 "R?" V 4680 3450 50  0000 C CNN
-F 1 "R" V 4600 3450 50  0000 C CNN
-F 2 "" V 4530 3450 50  0001 C CNN
-F 3 "" H 4600 3450 50  0001 C CNN
-	1    4600 3450
-	0    1    1    0
+P 4050 4000
+F 0 "R?" V 4130 4000 50  0000 C CNN
+F 1 "100K" V 4050 4000 50  0000 C CNN
+F 2 "" V 3980 4000 50  0001 C CNN
+F 3 "" H 4050 4000 50  0001 C CNN
+	1    4050 4000
+	-1   0    0    1
 $EndComp
 $Comp
 L R R?
 U 1 1 5AA9E04C
-P 4600 3150
-F 0 "R?" V 4680 3150 50  0000 C CNN
-F 1 "R" V 4600 3150 50  0000 C CNN
-F 2 "" V 4530 3150 50  0001 C CNN
-F 3 "" H 4600 3150 50  0001 C CNN
-	1    4600 3150
-	0    1    1    0
+P 4550 3100
+F 0 "R?" V 4630 3100 50  0000 C CNN
+F 1 "100K" V 4550 3100 50  0000 C CNN
+F 2 "" V 4480 3100 50  0001 C CNN
+F 3 "" H 4550 3100 50  0001 C CNN
+	1    4550 3100
+	-1   0    0    1
 $EndComp
 $Comp
 L R R?
 U 1 1 5AA9E082
-P 4600 2850
-F 0 "R?" V 4680 2850 50  0000 C CNN
-F 1 "R" V 4600 2850 50  0000 C CNN
-F 2 "" V 4530 2850 50  0001 C CNN
-F 3 "" H 4600 2850 50  0001 C CNN
-	1    4600 2850
-	0    1    1    0
-$EndComp
-Wire Wire Line
-	4750 3750 4900 3750
-Wire Wire Line
-	4900 3450 4750 3450
-Wire Wire Line
-	4750 3150 4900 3150
-Wire Wire Line
-	4750 2850 4900 2850
+P 4350 3100
+F 0 "R?" V 4430 3100 50  0000 C CNN
+F 1 "1K" V 4350 3100 50  0000 C CNN
+F 2 "" V 4280 3100 50  0001 C CNN
+F 3 "" H 4350 3100 50  0001 C CNN
+	1    4350 3100
+	-1   0    0    1
+$EndComp
 $Comp
 L R R?
@@
 P 4600 4050
 F 0 "R?" V 4680 4050 50  0000 C CNN
-F 1 "R" V 4600 4050 50  0000 C CNN
+F 1 "100K" V 4600 4050 50  0000 C CNN
 F 2 "" V 4530 4050 50  0001 C CNN
 F 3 "" H 4600 4050 50  0001 C CNN
@@
 $EndComp
 Wire Wire Line
-	4100 3750 4450 3750
-Wire Wire Line
 	4300 4050 4300 4650
 $Comp
@@
 P 4600 4500
 F 0 "R?" V 4680 4500 50  0000 C CNN
-F 1 "R" V 4600 4500 50  0000 C CNN
+F 1 "20K" V 4600 4500 50  0000 C CNN
 F 2 "" V 4530 4500 50  0001 C CNN
 F 3 "" H 4600 4500 50  0001 C CNN
@@
 L +3V3 #PWR?
 U 1 1 5AA9EC5E
-P 3750 2750
-F 0 "#PWR?" H 3750 2600 50  0001 C CNN
-F 1 "+3V3" H 3750 2890 50  0000 C CNN
-F 2 "" H 3750 2750 50  0001 C CNN
-F 3 "" H 3750 2750 50  0001 C CNN
-	1    3750 2750
-	1    0    0    -1
-$EndComp
-Wire Wire Line
-	4200 3450 4450 3450
+P 4450 2750
+F 0 "#PWR?" H 4450 2600 50  0001 C CNN
+F 1 "+3V3" H 4450 2890 50  0000 C CNN
+F 2 "" H 4450 2750 50  0001 C CNN
+F 3 "" H 4450 2750 50  0001 C CNN
+	1    4450 2750
+	1    0    0    -1
+$EndComp
 $Comp
 L C C?
@@
 P 4450 2350
 F 0 "C?" H 4475 2450 50  0000 L CNN
-F 1 "C" H 4475 2250 50  0000 L CNN
+F 1 "0.47u" H 4475 2250 50  0000 L CNN
 F 2 "" H 4488 2200 50  0001 C CNN
 F 3 "" H 4450 2350 50  0001 C CNN
@@
 P 5250 1400
 F 0 "C?" H 5275 1500 50  0000 L CNN
-F 1 "C" H 5275 1300 50  0000 L CNN
+F 1 "0.47u" H 5275 1300 50  0000 L CNN
 F 2 "" H 5288 1250 50  0001 C CNN
 F 3 "" H 5250 1400 50  0001 C CNN
@@
 P 5100 1900
 F 0 "C?" H 5125 2000 50  0000 L CNN
-F 1 "C" H 5125 1800 50  0000 L CNN
+F 1 "0.1u" H 5125 1800 50  0000 L CNN
 F 2 "" H 5138 1750 50  0001 C CNN
 F 3 "" H 5100 1900 50  0001 C CNN
@@
 P 5850 1400
 F 0 "C?" H 5875 1500 50  0000 L CNN
-F 1 "C" H 5875 1300 50  0000 L CNN
+F 1 "0.47u" H 5875 1300 50  0000 L CNN
 F 2 "" H 5888 1250 50  0001 C CNN
 F 3 "" H 5850 1400 50  0001 C CNN
@@
 P 5700 1850
 F 0 "C?" H 5725 1950 50  0000 L CNN
-F 1 "C" H 5725 1750 50  0000 L CNN
+F 1 "0.1u" H 5725 1750 50  0000 L CNN
 F 2 "" H 5738 1700 50  0001 C CNN
 F 3 "" H 5700 1850 50  0001 C CNN
@@
 P 6600 1550
 F 0 "C?" H 6625 1650 50  0000 L CNN
-F 1 "C" H 6625 1450 50  0000 L CNN
+F 1 "0.47u" H 6625 1450 50  0000 L CNN
 F 2 "" H 6638 1400 50  0001 C CNN
 F 3 "" H 6600 1550 50  0001 C CNN
@@
 P 6400 1850
 F 0 "C?" H 6425 1950 50  0000 L CNN
-F 1 "C" H 6425 1750 50  0000 L CNN
+F 1 "0.1u" H 6425 1750 50  0000 L CNN
 F 2 "" H 6438 1700 50  0001 C CNN
 F 3 "" H 6400 1850 50  0001 C CNN
@@
 L CONN_01X04 J?
 U 1 1 5AAA1490
-P 3650 3500
-F 0 "J?" H 3650 3750 50  0000 C CNN
-F 1 "CONN_01X04" V 3750 3500 50  0000 C CNN
-F 2 "" H 3650 3500 50  0001 C CNN
-F 3 "" H 3650 3500 50  0001 C CNN
-	1    3650 3500
+P 3800 3500
+F 0 "J?" H 3800 3750 50  0000 C CNN
+F 1 "CONN_01X04" V 3900 3500 50  0000 C CNN
+F 2 "" H 3800 3500 50  0001 C CNN
+F 3 "" H 3800 3500 50  0001 C CNN
+	1    3800 3500
 	-1   0    0    -1
 $EndComp
@@
 	4450 4050 4300 4050
 Wire Wire Line
-	4100 3750 4100 3650
-Wire Wire Line
-	4100 3650 3850 3650
-Wire Wire Line
-	4200 3450 4200 3550
-Wire Wire Line
-	4200 3550 3850 3550
-Wire Wire Line
-	4450 3150 4450 3300
-Wire Wire Line
-	4450 3300 4100 3300
-Wire Wire Line
-	4100 3300 4100 3450
-Wire Wire Line
-	4100 3450 3850 3450
-Wire Wire Line
-	4450 2850 4000 2850
-Wire Wire Line
-	4000 2850 4000 3350
-Wire Wire Line
-	4000 3350 3850 3350
-Wire Wire Line
-	3750 2750 4350 2750
-Wire Wire Line
-	4350 2750 4350 2850
-Connection ~ 4350 2850
-Wire Wire Line
-	4300 3300 4300 2750
-Connection ~ 4300 2750
-Connection ~ 4300 3300
-Wire Wire Line
-	4150 3550 4150 2750
-Connection ~ 4150 2750
-Connection ~ 4150 3550
-Wire Wire Line
-	3950 3650 3950 2750
-Connection ~ 3950 2750
-Connection ~ 3950 3650
+	4000 3550 4900 3550
+Wire Wire Line
+	4000 3450 4900 3450
+Wire Wire Line
+	4000 3350 4900 3350
 $Comp
 L CONN_01X01 J?
@@
 L Screw_Terminal_1x02 J?
 U 1 1 5AAA2A35
-P 8450 3750
-F 0 "J?" H 8450 4000 50  0000 C TNN
-F 1 "Screw_Terminal_1x02" V 8300 3750 50  0000 C TNN
-F 2 "" H 8450 3525 50  0001 C CNN
-F 3 "" H 8425 3750 50  0001 C CNN
-	1    8450 3750
+P 8250 1350
+F 0 "J?" H 8250 1600 50  0000 C TNN
+F 1 "Screw_Terminal_1x02" V 8100 1350 50  0000 C TNN
+F 2 "" H 8250 1125 50  0001 C CNN
+F 3 "" H 8225 1350 50  0001 C CNN
+	1    8250 1350
 	-1   0    0    -1
 $EndComp
@@
 L +3V3 #PWR?
 U 1 1 5AAA316A
-P 8050 3400
-F 0 "#PWR?" H 8050 3250 50  0001 C CNN
-F 1 "+3V3" H 8050 3540 50  0000 C CNN
-F 2 "" H 8050 3400 50  0001 C CNN
-F 3 "" H 8050 3400 50  0001 C CNN
-	1    8050 3400
+P 7850 1000
+F 0 "#PWR?" H 7850 850 50  0001 C CNN
+F 1 "+3V3" H 7850 1140 50  0000 C CNN
+F 2 "" H 7850 1000 50  0001 C CNN
+F 3 "" H 7850 1000 50  0001 C CNN
+	1    7850 1000
 	1    0    0    -1
 $EndComp
@@
 L GND #PWR?
 U 1 1 5AAA3289
-P 8050 4000
-F 0 "#PWR?" H 8050 3750 50  0001 C CNN
-F 1 "GND" H 8050 3850 50  0000 C CNN
-F 2 "" H 8050 4000 50  0001 C CNN
-F 3 "" H 8050 4000 50  0001 C CNN
-	1    8050 4000
-	1    0    0    -1
-$EndComp
-Wire Wire Line
-	8250 3650 8050 3650
-Wire Wire Line
-	8050 3650 8050 3400
-Wire Wire Line
-	8250 3850 8050 3850
-Wire Wire Line
-	8050 3850 8050 4000
+P 7850 1600
+F 0 "#PWR?" H 7850 1350 50  0001 C CNN
+F 1 "GND" H 7850 1450 50  0000 C CNN
+F 2 "" H 7850 1600 50  0001 C CNN
+F 3 "" H 7850 1600 50  0001 C CNN
+	1    7850 1600
+	1    0    0    -1
+$EndComp
+Wire Wire Line
+	8050 1250 7850 1250
+Wire Wire Line
+	7850 1250 7850 1000
+Wire Wire Line
+	8050 1450 7850 1450
+Wire Wire Line
+	7850 1450 7850 1600
+Wire Wire Line
+	4550 3250 4550 3550
+Connection ~ 4550 3550
+Wire Wire Line
+	4350 3250 4350 3450
+Connection ~ 4350 3450
+Wire Wire Line
+	4150 3250 4150 3350
+Connection ~ 4150 3350
+Wire Wire Line
+	4150 2950 4150 2850
+Wire Wire Line
+	4150 2850 4550 2850
+Wire Wire Line
+	4350 2850 4350 2950
+Connection ~ 4350 2850
+Wire Wire Line
+	4550 2850 4550 2950
+Wire Wire Line
+	4450 2850 4450 2750
+Connection ~ 4450 2850
+Wire Wire Line
+	4900 3650 4000 3650
+Wire Wire Line
+	4050 3850 4050 3650
+Connection ~ 4050 3650
+$Comp
+L GND #PWR?
+U 1 1 5AAA5323
+P 4050 4250
+F 0 "#PWR?" H 4050 4000 50  0001 C CNN
+F 1 "GND" H 4050 4100 50  0000 C CNN
+F 2 "" H 4050 4250 50  0001 C CNN
+F 3 "" H 4050 4250 50  0001 C CNN
+	1    4050 4250
+	1    0    0    -1
+$EndComp
+Wire Wire Line
+	4050 4150 4050 4250
 $EndSCHEMATC

Commit message: [ci skip] Annotate schematic components
Parts:
- gave numbers to parts that had none: 23
Changed lines of the file:
@@
 $EndDescr
 $Comp
-L IS31FL3733 U?
+L IS31FL3733 U1
 U 1 1 5AA9A71C
 P 5900 4150
-F 0 "U?" H 5900 5000 60  0000 C CNN
+F 0 "U1" H 5900 5000 60  0000 C CNN
 F 1 "IS31FL3733" H 5900 4850 60  0000 C CNN
 F 2 "" H 5900 4850 60  0001 C CNN
@@
 $EndComp
 $Comp
-L CONN_01X12 J?
+L CONN_01X12 J4
 U 1 1 5AA9B2E6
 P 7250 4650
-F 0 "J?" H 7250 5300 50  0000 C CNN
+F 0 "J4" H 7250 5300 50  0000 C CNN
 F 1 "CONN_01X12" V 7350 4650 50  0000 C CNN
 F 2 "" H 7250 4650 50  0001 C CNN
@@
 $EndComp
 $Comp
-L CONN_01X16 J?
+L CONN_01X16 J3
 U 1 1 5AA9B36B
 P 7250 3150
-F 0 "J?" H 7250 4000 50  0000 C CNN
+F 0 "J3" H 7250 4000 50  0000 C CNN
 F 1 "CONN_01X16" V 7350 3150 50  0000 C CNN
 F 2 "" H 7250 3150 50  0001 C CNN
@@
 	6950 5200 7050 5200
 $Comp
-L R R?
+L R R9
 U 1 1 5AA9C11D
 P 4700 5150
-F 0 "R?" V 4780 5150 50  0000 C CNN
+F 0 "R9" V 4780 5150 50  0000 C CNN
 F 1 "0" V 4700 5150 50  0000 C CNN
 F 2 "" V 4630 5150 50  0001 C CNN
@@
 $EndComp
 $Comp
-L R R?
+L R R10
 U 1 1 5AA9C30E
 P 4700 5500
-F 0 "R?" V 4780 5500 50  0000 C CNN
+F 0 "R10" V 4780 5500 50  0000 C CNN
 F 1 "0" V 4700 5500 50  0000 C CNN
 F 2 "" V 4630 5500 50  0001 C CNN
@@
 	4850 5500 4900 5500
 $Comp
-L +3V3 #PWR?
+L +3V3 #PWR3
 U 1 1 5AA9C5FA
 P 4050 5000
-F 0 "#PWR?" H 4050 4850 50  0001 C CNN
+F 0 "#PWR3" H 4050 4850 50  0001 C CNN
 F 1 "+3V3" H 4050 5140 50  0000 C CNN
 F 2 "" H 4050 5000 50  0001 C CNN
@@
 $EndComp
 $Comp
-L R R?
+L R R3
 U 1 1 5AA9C6C1
 P 4300 5150
-F 0 "R?" V 4380 5150 50  0000 C CNN
+F 0 "R3" V 4380 5150 50  0000 C CNN
 F 1 "0" V 4300 5150 50  0000 C CNN
 F 2 "" V 4230 5150 50  0001 C CNN
@@
 $EndComp
 $Comp
-L R R?
+L R R4
 U 1 1 5AA9C6FF
 P 4300 5500
-F 0 "R?" V 4380 5500 50  0000 C CNN
+F 0 "R4" V 4380 5500 50  0000 C CNN
 F 1 "0" V 4300 5500 50  0000 C CNN
 F 2 "" V 4230 5500 50  0001 C CNN
@@
 	4450 5500 4550 5500
 $Comp
-L GND #PWR?
+L GND #PWR7
 U 1 1 5AA9CCBA
 P 4500 5600
-F 0 "#PWR?" H 4500 5350 50  0001 C CNN
+F 0 "#PWR7" H 4500 5350 50  0001 C CNN
 F 1 "GND" H 4500 5450 50  0000 C CNN
 F 2 "" H 4500 5600 50  0001 C CNN
@@
 $EndComp
 $Comp
-L GND #PWR?
+L GND #PWR6
 U 1 1 5AA9CE00
 P 4500 5250
-F 0 "#PWR?" H 4500 5000 50  0001 C CNN
+F 0 "#PWR6" H 4500 5000 50  0001 C CNN
 F 1 "GND" H 4500 5100 50  0000 C CNN
 F 2 "" H 4500 5250 50  0001 C CNN
@@
 Connection ~ 4050 5150
 $Comp
-L +3V3 #PWR?
+L +3V3 #PWR8
 U 1 1 5AA9D8F8
 P 4750 2200
-F 0 "#PWR?" H 4750 2050 50  0001 C CNN
+F 0 "#PWR8" H 4750 2050 50  0001 C CNN
 F 1 "+3V3" H 4750 2340 50  0000 C CNN
 F 2 "" H 4750 2200 50  0001 C CNN
@@
 $EndComp
 $Comp
-L GND #PWR?
+L GND #PWR1
 U 1 1 5AA9DBD7
 P 3950 2400
-F 0 "#PWR?" H 3950 2150 50  0001 C CNN
+F 0 "#PWR1" H 3950 2150 50  0001 C CNN
 F 1 "GND" H 3950 2250 50  0000 C CNN
 F 2 "" H 3950 2400 50  0001 C CNN
@@
 $EndComp
 $Comp
-L R R?
+L R R2
 U 1 1 5AA9DEC1
 P 4150 3100
-F 0 "R?" V 4230 3100 50  0000 C CNN
+F 0 "R2" V 4230 3100 50  0000 C CNN
 F 1 "1K" V 4150 3100 50  0000 C CNN
 F 2 "" V 4080 3100 50  0001 C CNN
@@
 $EndComp
 $Comp
-L R R?
+L R R1
 U 1 1 5AA9E017
 P 4050 4000
-F 0 "R?" V 4130 4000 50  0000 C CNN
+F 0 "R1" V 4130 4000 50  0000 C CNN
 F 1 "100K" V 4050 4000 50  0000 C CNN
 F 2 "" V 3980 4000 50  0001 C CNN
@@
 $EndComp
 $Comp
-L R R?
+L R R6
 U 1 1 5AA9E04C
 P 4550 3100
-F 0 "R?" V 4630 3100 50  0000 C CNN
+F 0 "R6" V 4630 3100 50  0000 C CNN
 F 1 "100K" V 4550 3100 50  0000 C CNN
 F 2 "" V 4480 3100 50  0001 C CNN
@@
 $EndComp
 $Comp
-L R R?
+L R R5
 U 1 1 5AA9E082
 P 4350 3100
-F 0 "R?" V 4430 3100 50  0000 C CNN
+F 0 "R5" V 4430 3100 50  0000 C CNN
 F 1 "1K" V 4350 3100 50  0000 C CNN
 F 2 "" V 4280 3100 50  0001 C CNN
@@
 $EndComp
 $Comp
-L R R?
+L R R7
 U 1 1 5AA9E531
 P 4600 4050
-F 0 "R?" V 4680 4050 50  0000 C CNN
+F 0 "R7" V 4680 4050 50  0000 C CNN
 F 1 "100K" V 4600 4050 50  0000 C CNN
 F 2 "" V 4530 4050 50  0001 C CNN
@@
 	4750 4050 4900 4050
 $Comp
-L GND #PWR?
+L GND #PWR4
 U 1 1 5AA9E6FB
 P 4300 4650
-F 0 "#PWR?" H 4300 4400 50  0001 C CNN
+F 0 "#PWR4" H 4300 4400 50  0001 C CNN
 F 1 "GND" H 4300 4500 50  0000 C CNN
 F 2 "" H 4300 4650 50  0001 C CNN
@@
 	4300 4050 4300 4650
 $Comp
-L R R?
+L R R8
 U 1 1 5AA9E9E1
 P 4600 4500
-F 0 "R?" V 4680 4500 50  0000 C CNN
+F 0 "R8" V 4680 4500 50  0000 C CNN
 F 1 "20K" V 4600 4500 50  0000 C CNN
 F 2 "" V 4530 4500 50  0001 C CNN
@@
 Connection ~ 4300 4500
 $Comp
-L +3V3 #PWR?
+L +3V3 #PWR5
 U 1 1 5AA9EC5E
 P 4450 2750
-F 0 "#PWR?" H 4450 2600 50  0001 C CNN
+F 0 "#PWR5" H 4450 2600 50  0001 C CNN
 F 1 "+3V3" H 4450 2890 50  0000 C CNN
 F 2 "" H 4450 2750 50  0001 C CNN
@@
 $EndComp
 $Comp
-L C C?
+L C C1
 U 1 1 5AA9EDEF
 P 4450 2350
-F 0 "C?" H 4475 2450 50  0000 L CNN
+F 0 "C1" H 4475 2450 50  0000 L CNN
 F 1 "0.47u" H 4475 2250 50  0000 L CNN
 F 2 "" H 4488 2200 50  0001 C CNN
@@
 	3950 2350 3950 2400
 $Comp
-L GND #PWR?
+L GND #PWR14
 U 1 1 5AA9F4CE
 P 5900 6350
-F 0 "#PWR?" H 5900 6100 50  0001 C CNN
+F 0 "#PWR14" H 5900 6100 50  0001 C CNN
 F 1 "GND" H 5900 6200 50  0000 C CNN
 F 2 "" H 5900 6350 50  0001 C CNN
@@
 Connection ~ 6350 6250
 $Comp
-L +3V3 #PWR?
+L +3V3 #PWR11
 U 1 1 5AA9FB8D
 P 5450 1150
-F 0 "#PWR?" H 5450 1000 50  0001 C CNN
+F 0 "#PWR11" H 5450 1000 50  0001 C CNN
 F 1 "+3V3" H 5450 1290 50  0000 C CNN
 F 2 "" H 5450 1150 50  0001 C CNN
@@
 $EndComp
 $Comp
-L +3V3 #PWR?
+L +3V3 #PWR15
 U 1 1 5AA9FE0E
 P 6100 1350
-F 0 "#PWR?" H 6100 1200 50  0001 C CNN
+F 0 "#PWR15" H 6100 1200 50  0001 C CNN
 F 1 "+3V3" H 6100 1490 50  0000 C CNN
 F 2 "" H 6100 1350 50  0001 C CNN
@@
 $EndComp
 $Comp
-L C C?
+L C C3
 U 1 1 5AA9FE43
 P 5250 1400
-F 0 "C?" H 5275 1500 50  0000 L CNN
+F 0 "C3" H 5275 1500 50  0000 L CNN
 F 1 "0.47u" H 5275 1300 50  0000 L CNN
 F 2 "" H 5288 1250 50  0001 C CNN
@@
 $EndComp
 $Comp
-L C C?
+L C C2
 U 1 1 5AA9FEB6
 P 5100 1900
-F 0 "C?" H 5125 2000 50  0000 L CNN
+F 0 "C2" H 5125 2000 50  0000 L CNN
 F 1 "0.1u" H 5125 1800 50  0000 L CNN
 F 2 "" H 5138 1750 50  0001 C CNN
@@
 $EndComp
 $Comp
-L C C?
+L C C5
 U 1 1 5AA9FEFE
 P 5850 1400
-F 0 "C?" H 5875 1500 50  0000 L CNN
+F 0 "C5" H 5875 1500 50  0000 L CNN
 F 1 "0.47u" H 5875 1300 50  0000 L CNN
 F 2 "" H 5888 1250 50  0001 C CNN
@@
 $EndComp
 $Comp
-L C C?
+L C C4
 U 1 1 5AA9FF59
 P 5700 1850
-F 0 "C?" H 5725 1950 50  0000 L CNN
+F 0 "C4" H 5725 1950 50  0000 L CNN
 F 1 "0.1u" H 5725 1750 50  0000 L CNN
 F 2 "" H 5738 1700 50  0001 C CNN
@@
 Connection ~ 5550 1700
 $Comp
-L GND #PWR?
+L GND #PWR13
 U 1 1 5AAA086A
 P 5850 1550
-F 0 "#PWR?" H 5850 1300 50  0001 C CNN
+F 0 "#PWR13" H 5850 1300 50  0001 C CNN
 F 1 "GND" H 5850 1400 50  0000 C CNN
 F 2 "" H 5850 1550 50  0001 C CNN
@@
 $EndComp
 $Comp
-L GND #PWR?
+L GND #PWR12
 U 1 1 5AAA0A6D
 P 5700 2000
-F 0 "#PWR?" H 5700 1750 50  0001 C CNN
+F 0 "#PWR12" H 5700 1750 50  0001 C CNN
 F 1 "GND" H 5700 1850 50  0000 C CNN
 F 2 "" H 5700 2000 50  0001 C CNN
@@
 $EndComp
 $Comp
-L GND #PWR?
+L GND #PWR9
 U 1 1 5AAA0AC0
 P 5100 2050
-F 0 "#PWR?" H 5100 1800 50  0001 C CNN
+F 0 "#PWR9" H 5100 1800 50  0001 C CNN
 F 1 "GND" H 5100 1900 50  0000 C CNN
 F 2 "" H 5100 2050 50  0001 C CNN
@@
 $EndComp
 $Comp
-L GND #PWR?
+L GND #PWR10
 U 1 1 5AAA0B01
 P 5250 1550
-F 0 "#PWR?" H 5250 1300 50  0001 C CNN
+F 0 "#PWR10" H 5250 1300 50  0001 C CNN
 F 1 "GND" H 5250 1400 50  0000 C CNN
 F 2 "" H 5250 1550 50  0001 C CNN
@@
 Connection ~ 6100 1950
 $Comp
-L C C?
+L C C7
 U 1 1 5AAA0C1D
 P 6600 1550
-F 0 "C?" H 6625 1650 50  0000 L CNN
+F 0 "C7" H 6625 1650 50  0000 L CNN
 F 1 "0.47u" H 6625 1450 50  0000 L CNN
 F 2 "" H 6638 1400 50  0001 C CNN
@@
 $EndComp
 $Comp
-L C C?
+L C C6
 U 1 1 5AAA0C88
 P 6400 1850
-F 0 "C?" H 6425 1950 50  0000 L CNN
+F 0 "C6" H 6425 1950 50  0000 L CNN
 F 1 "0.1u" H 6425 1750 50  0000 L CNN
 F 2 "" H 6438 1700 50  0001 C CNN
@@
 Connection ~ 6100 1400
 $Comp
-L GND #PWR?
+L GND #PWR16
 U 1 1 5AAA0F04
 P 6400 2000
-F 0 "#PWR?" H 6400 1750 50  0001 C CNN
+F 0 "#PWR16" H 6400 1750 50  0001 C CNN
 F 1 "GND" H 6400 1850 50  0000 C CNN
 F 2 "" H 6400 2000 50  0001 C CNN
@@
 $EndComp
 $Comp
-L GND #PWR?
+L GND #PWR17
 U 1 1 5AAA0F4B
 P 6600 1700
-F 0 "#PWR?" H 6600 1450 50  0001 C CNN
+F 0 "#PWR17" H 6600 1450 50  0001 C CNN
 F 1 "GND" H 6600 1550 50  0000 C CNN
 F 2 "" H 6600 1700 50  0001 C CNN
@@
 $EndComp
 $Comp
-L CONN_01X04 J?
+L CONN_01X04 J2
 U 1 1 5AAA1490
 P 3800 3500
-F 0 "J?" H 3800 3750 50  0000 C CNN
+F 0 "J2" H 3800 3750 50  0000 C CNN
 F 1 "CONN_01X04" V 3900 3500 50  0000 C CNN
 F 2 "" H 3800 3500 50  0001 C CNN
@@
 	4000 3350 4900 3350
 $Comp
-L CONN_01X01 J?
+L CONN_01X01 J1
 U 1 1 5AAA24C9
 P 3450 4650
-F 0 "J?" H 3450 4750 50  0000 C CNN
+F 0 "J1" H 3450 4750 50  0000 C CNN
 F 1 "CONN_01X01" V 3550 4650 50  0000 C CNN
 F 2 "" H 3450 4650 50  0001 C CNN
@@
 	4200 4650 3650 4650
 $Comp
-L Screw_Terminal_1x02 J?
+L Screw_Terminal_1x02 J5
 U 1 1 5AAA2A35
 P 8250 1350
-F 0 "J?" H 8250 1600 50  0000 C TNN
+F 0 "J5" H 8250 1600 50  0000 C TNN
 F 1 "Screw_Terminal_1x02" V 8100 1350 50  0000 C TNN
 F 2 "" H 8250 1125 50  0001 C CNN
@@
 $EndComp
 $Comp
-L +3V3 #PWR?
+L +3V3 #PWR18
 U 1 1 5AAA316A
 P 7850 1000
-F 0 "#PWR?" H 7850 850 50  0001 C CNN
+F 0 "#PWR18" H 7850 850 50  0001 C CNN
 F 1 "+3V3" H 7850 1140 50  0000 C CNN
 F 2 "" H 7850 1000 50  0001 C CNN
@@
 $EndComp
 $Comp
-L GND #PWR?
+L GND #PWR19
 U 1 1 5AAA3289
 P 7850 1600
-F 0 "#PWR?" H 7850 1350 50  0001 C CNN
+F 0 "#PWR19" H 7850 1350 50  0001 C CNN
 F 1 "GND" H 7850 1450 50  0000 C CNN
 F 2 "" H 7850 1600 50  0001 C CNN
@@
 Connection ~ 4050 3650
 $Comp
-L GND #PWR?
+L GND #PWR2
 U 1 1 5AAA5323
 P 4050 4250
-F 0 "#PWR?" H 4050 4000 50  0001 C CNN
+F 0 "#PWR2" H 4050 4000 50  0001 C CNN
 F 1 "GND" H 4050 4100 50  0000 C CNN
 F 2 "" H 4050 4250 50  0001 C CNN
