File: hardware/kicad/matrix-dev/matrix-dev-board.sch (KiCad schematic (older format))
At the start: 23 parts, among them J1 CONN_01X01, J2 CONN_01X04, J3 CONN_01X16, J4 CONN_01X12, J5 Screw_Terminal_1x02, U1 IS31FL3733

Commit message: [ci skip] First attempt at laying out the matrix dev board
Parts:
- removed R3, R4: 0, symbol R
- C1, C2, C3, C4, C5, C6, C7: footprint (none) -> Capacitors_SMD:C_0805_HandSoldering
- J1: footprint (none) -> Pin_Headers:Pin_Header_Straight_1x01_Pitch1.27mm
- J2: footprint (none) -> Pin_Headers:Pin_Header_Angled_1x04_Pitch1.27mm
- J3: footprint (none) -> Pin_Headers:Pin_Header_Angled_1x16_Pitch1.27mm
- J4: footprint (none) -> Pin_Headers:Pin_Header_Angled_1x12_Pitch1.27mm
- J5: footprint (none) -> Pin_Headers:Pin_Header_Straight_1x02_Pitch2.54mm
- R1, R10, R2, R5, R6, R7, R8, R9: footprint (none) -> Resistors_SMD:R_0805_HandSoldering
- U1: footprint (none) -> Housings_DFN_QFN:QFN-48-1EP_6x6mm_Pitch0.4mm_ThermalVias
Connections:
- net at U1.10 (SW8): now also J4.5 (P5); no longer J4.8 (P8)
- net at U1.11 (SW9): now also J4.4 (P4); no longer J4.9 (P9)
- net at U1.13 (SW10): now also J4.3 (P3); no longer J4.10 (P10)
- net at U1.14 (SW11): now also J4.2 (P2); no longer J4.11 (P11)
- net at U1.15 (SW12): now also J4.1 (P1); no longer J4.12 (P12)
- net at U1.16 (CS1): now also J3.16 (P16); no longer J3.1 (P1)
- net at U1.17 (CS2): now also J3.15 (P15); no longer J3.2 (P2)
- net at U1.18 (CS3): now also J3.14 (P14); no longer J3.3 (P3)
- net at U1.19 (CS4): now also J3.13 (P13); no longer J3.4 (P4)
- net at U1.2 (SW1): now also J4.12 (P12); no longer J4.1 (P1)
- net at U1.21 (CS5): now also J3.12 (P12); no longer J3.5 (P5)
- net at U1.22 (CS6): now also J3.11 (P11); no longer J3.6 (P6)
- net at U1.23 (CS7): now also J3.10 (P10); no longer J3.7 (P7)
- net at U1.24 (CS8): now also J3.9 (P9); no longer J3.8 (P8)
- net at U1.25 (CS9): now also J3.8 (P8); no longer J3.9 (P9)
- net at U1.26 (CS10): now also J3.7 (P7); no longer J3.10 (P10)
- net at U1.27 (CS11): now also J3.6 (P6); no longer J3.11 (P11)
- net at U1.28 (CS12): now also J3.5 (P5); no longer J3.12 (P12)
- net at U1.3 (SW2): now also J4.11 (P11); no longer J4.2 (P2)
- net at U1.30 (CS13): now also J3.4 (P4); no longer J3.13 (P13)
- net at U1.31 (CS14): now also J3.3 (P3); no longer J3.14 (P14)
- net at U1.32 (CS15): now also J3.2 (P2); no longer J3.15 (P15)
- net at U1.33 (CS16): now also J3.1 (P1); no longer J3.16 (P16)
- net at U1.4 (SW3): now also J4.10 (P10); no longer J4.3 (P3)
- net at R2.1, U1.41 (SDA): now also J2.4 (P4); no longer J2.1 (P1)
- net at R5.1, U1.42 (SCL): now also J2.3 (P3); no longer J2.2 (P2)
- net at R6.1, U1.45 (INTB): now also J2.2 (P2); no longer J2.3 (P3)
- net at R1.2, U1.46 (SDB): now also J2.1 (P1); no longer J2.4 (P4)
- net at U1.6 (SW4): now also J4.9 (P9); no longer J4.4 (P4)
- net at U1.7 (SW5): now also J4.8 (P8); no longer J4.5 (P5)
- net at U1.8 (SW6): now also J4.7 (P7); no longer J4.6 (P6)
- net at U1.9 (SW7): now also J4.6 (P6); no longer J4.7 (P7)

Commit message: :memo: Add reference to datasheet and digikey page
Parts:
- U1: DKPN (none) -> 706-1509-1-ND
Changed lines of the file:
@@
 F 1 "IS31FL3733" H 5900 4850 60  0000 C CNN
 F 2 "Housings_DFN_QFN:QFN-48-1EP_6x6mm_Pitch0.4mm_ThermalVias" H 5900 4850 60  0001 C CNN
-F 3 "" H 5900 4850 60  0001 C CNN
+F 3 "http://www.issi.com/WW/pdf/31FL3733.pdf" H 5900 4850 60  0001 C CNN
+F 4 "706-1509-1-ND" H 5900 4150 60  0001 C CNN "DKPN"
 	1    5900 4150
 	1    0    0    -1
